File: Circuit/hd44780_backpack.kicad_pcb (KiCad board)
At the start: 2 copper layers, 98.4 x 60.3 mm, 20 parts, among them IC1 ATTINY84A-SS, P1 I2C, P10 GND, P2 ISCP, P3 A0, P4 A1, P5 A7, P6 8, P7 10, P8 SERIAL QA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

Commit message: Added github link to text on back of board
Other:
- board text added: "Controller for HD4470 Screen Designed by John Spencer, 2014 https://github.com/mage0r/HD44780_Backpack Version 1.3"
- board text removed: "Controller for HD4470 Screen Designed by John Spencer, 2014 Version 1.3"
Changed lines of the file:
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@@
     (links 49)
     (no_connects 0)
-    (area 12.249999 12.249999 110.750001 72.650001)
+    (area 11.996 11.196 110.829001 72.779001)
     (thickness 1.6)
     (drawings 9)
@@
     (18 B.Paste user)
     (19 F.Paste user)
-    (20 B.SilkS user)
+    (20 B.SilkS user hide)
     (21 F.SilkS user)
     (22 B.Mask user)
@@
     (pcbplotparams
       (layerselection 284196865)
-      (usegerberextensions true)
+      (usegerberextensions false)
       (excludeedgelayer true)
       (linewidth 0.150000)
@@
       (padsonsilk false)
       (subtractmaskfromsilk false)
-      (outputformat 1)
+      (outputformat 5)
       (mirror false)
       (drillshape 0)
@@
   (gr_line (start 12.3 72.6) (end 110.7 72.6) (angle 90) (layer Edge.Cuts) (width 0.1))
   (gr_line (start 12.3 12.4) (end 12.3 72.6) (angle 90) (layer Edge.Cuts) (width 0.1))
-  (gr_text "Controller for HD4470 Screen\nDesigned by John Spencer, 2014\nVersion 1.3" (at 52.2 35.85) (layer B.SilkS)
+  (gr_text "Controller for HD4470 Screen\nDesigned by John Spencer, 2014\nhttps://github.com/mage0r/HD44780_Backpack\nVersion 1.3" (at 52.3 22.4) (layer B.SilkS)
     (effects (font (size 1.5 1.5) (thickness 0.3)) (justify mirror))
   )

Commit message: non-working circuit.
Parts:
- removed P10: GND, 1pin
- removed P9: +5V, 1pin
- added M1: MESHTHING, xbee_r1-XBEE, F.Cu at (33.1, 33.3)
- added PROTO_6X11: Z2, PROTO_6x11, F.Cu at (53.0, 30.7)
- added PROTO_6X11_2: Z1, PROTO_6x11, F.Cu at (33.4, 30.8)
- added R3: 10k, SM0805, F.Cu at (77.2, 42.1)
- P3: value A0 -> ATTINY_BREAKOUT; footprint 1pin -> ATtiny_breakout
- P4: value A1 -> POWER; footprint 1pin -> USB_MINI_B
- P5: value A7 -> CONN_10; footprint 1pin -> PIN_ARRAY_10X1
- P6: value 8 -> CONN_10; footprint 1pin -> PIN_ARRAY_10X1
- P7: value 10 -> CONN_4; footprint 1pin -> PIN_ARRAY_4x1
- P8: value SERIAL QA -> CONN_4X2; footprint PIN_ARRAY_1 -> pin_array_4x2
- moved P4 88.3 mm to (103.7, 25.1)
- moved 10k1 62.4 mm to (87.7, 23.3), turned to 90 degrees
- moved Q1 54.0 mm to (80.8, 28.7)
- moved R1 54.0 mm to (79.9, 31.8)
- moved P7 53.5 mm to (68.8, 45.5), turned to 90 degrees
- moved R2 51.9 mm to (82.6, 31.9), turned to 90 degrees
- moved C1 51.6 mm to (81.3, 23.3), turned to 0 degrees
- moved C2 51.6 mm to (81.3, 21.3), turned to 0 degrees
- moved P3 50.3 mm to (62.7, 38.3), turned to 270 degrees
- moved P8 29.6 mm to (72.7, 45.5), turned to 90 degrees
- moved P6 26.8 mm to (42.2, 35.7), turned to 270 degrees
- moved U1 13.9 mm to (71.7, 25.5)
- moved IC1 13.1 mm to (71.5, 35.6)
- moved P5 10.2 mm to (24.6, 35.7), turned to 90 degrees
- moved SW1 5.42 mm to (89.0, 31.1), turned to 180 degrees
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Connections:
- IC1 pad 10: N-0000017 -> N-0000018
- IC1 pad 11: N-0000018 -> N-0000043
- IC1 pad 12: N-000005 -> N-0000012
- IC1 pad 2: N-000007 -> N-0000045
- IC1 pad 3: N-0000012 -> N-0000044
- IC1 pad 5: N-000006 -> N-0000010
- IC1 pad 6: N-000008 -> N-0000011
- IC1 pad 7: N-0000023 -> N-0000046
- IC1 pad 9: N-0000032 -> N-0000014
- P1 pad 1: N-0000023 -> N-0000046
- P1 pad 2: N-0000032 -> N-0000014
- P2 pad 3: N-0000032 -> N-0000014
- P2 pad 4: N-0000023 -> N-0000046
- P4 pad 1: N-000005 -> +5V
- P5 pad 1: N-000008 -> GND
- P6 pad 1: N-000006 -> N-0000015
- P7 pad 1: N-000007 -> N-0000015
- P8 pad 1: N-000004 -> N-0000045
- R1 pad 1: N-0000014 -> N-0000016
- U1 pad 11: N-0000017 -> N-0000021
- U1 pad 12: N-0000012 -> N-0000020
- U1 pad 14: N-0000018 -> N-0000017
- U1 pad 15: N-000004 -> (no net)
- U1 pad 2: N-0000014 -> (no net)
- U1 pad 4: N-0000020 -> N-0000022
- U1 pad 5: N-0000029 -> N-0000048
- U1 pad 6: N-0000030 -> N-0000049
- U1 pad 7: N-0000031 -> N-0000042
- U2 pad 11: N-0000020 -> N-0000042
- U2 pad 12: N-0000029 -> N-0000049
- U2 pad 13: N-0000030 -> N-0000048
- U2 pad 14: N-0000031 -> N-0000022
Routing:
- net GND: track 189.8 -> 0.00 mm
- net +5V: track 151.7 -> 0.00 mm, vias 2 -> 0
- net N-000008: track 68.1 -> 0.00 mm
- net N-000007: track 60.9 -> 0.00 mm
- net N-0000032: track 57.4 -> 0.00 mm
- net N-000006: track 54.7 -> 0.00 mm
- net N-000005: track 52.7 -> 0.00 mm, vias 1 -> 0
- net N-0000035: track 52.4 -> 0.00 mm, vias 1 -> 0
- net N-0000052: track 46.3 -> 0.00 mm
- net N-0000023: track 43.6 -> 0.00 mm
- net N-0000047: track 36.1 -> 0.00 mm
- net N-0000024: track 32.2 -> 0.00 mm
- net N-0000014: track 30.4 -> 0.00 mm
- net N-0000034: track 29.6 -> 0.00 mm
- net N-0000041: track 29.3 -> 0.00 mm
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Other:
- board text added: "Controller for HD4470 Screen Designed by John Spencer, 2014 https://github.com/mage0r/HD44780_Backpack Version 1.4 - Meshthingy Version"
- board text removed: "Controller for HD4470 Screen Designed by John Spencer, 2014 https://github.com/mage0r/HD44780_Backpack Version 1.3"

Commit message: Meshthing integration complete
Parts:
- added K1: PWR_SHIFT, PIN_ARRAY_3X1, F.Cu at (72.1, 39.1)
- added P9: CONN_2, PIN_ARRAY_2X1, F.Cu at (62.7, 40.9)
- added Q2: BSS138, SOT23, F.Cu at (76.3, 21.7)
- added Q3: BSS138, SOT23, F.Cu at (72.9, 17.6)
- added R4: 10K, SM0805, F.Cu at (79.4, 19.3)
- added R5: 10K, SM0805, F.Cu at (76.3, 24.6)
- added R6: 10K, SM0805, F.Cu at (72.4, 14.2)
- added R7: 10K, SM0805, F.Cu at (75.7, 17.6)
- added R8: 1K, SM0805, F.Cu at (21.4, 19.4)
- added R9: 2.2K, SM0805, F.Cu at (19.4, 19.4)
- P4: value POWER -> USB_5PIN_SHELL; footprint USB_MINI_B -> MINI_USB
- P5: value CONN_10 -> MESH_BKOUT_1-10
- P6: value CONN_10 -> MESH_BKOUT_11-20
- P7: value CONN_4 -> MESH_ENABLE
- P8: value CONN_4X2 -> ATTINY_ENABLE
- moved P4 21.7 mm to (84.5, 14.9)
- moved R3 8.15 mm to (71.1, 36.7)
- moved U1 7.37 mm to (66.8, 20.0)
- moved P3 5.00 mm to (62.7, 33.3)
- moved IC1 4.90 mm to (71.3, 30.7)
- moved P1 3.54 mm to (76.8, 14.0)
- moved P5 3.01 mm to (21.6, 35.4)
- moved P6 3.01 mm to (39.2, 35.4)
- moved M1 3.01 mm to (30.1, 33.0)
- moved PROTO_6X11_2 3.01 mm to (30.4, 30.5)
- moved P7 0.70 mm to (69.5, 45.5)
- moved P8 0.70 mm to (73.4, 45.5)
- moved P2 0.40 mm to (82.4, 39.5)
Connections:
- IC1 pad 7: N-0000046 (its old number) -> N-0000032
- IC1 pad 9: N-0000014 (its old number) -> N-0000019
- M1 pad 1: N-0000027 (its old number) -> +3.3V
- M1 pad 13: N-0000014 (its old number) -> N-0000022
- M1 pad 9: N-0000046 (its old number) -> N-0000033
- P1 pad 1: N-0000046 (its old number) -> N-0000032
- P1 pad 2: N-0000014 (its old number) -> N-0000019
- P2 pad 3: N-0000014 (its old number) -> N-0000019
- P2 pad 4: N-0000046 (its old number) -> N-0000032
- P4 pad 2: GND -> (no net)
- P4 pad 5: (no net) -> GND
- P5 pad 10: N-0000027 (its old number) -> +3.3V
- P5 pad 2: N-0000046 (its old number) -> N-0000033
- P6 pad 8: N-0000014 (its old number) -> N-0000022
- R3 pad 2: +5V -> N-0000060
- U1 pad 10: +5V -> N-0000060
- U1 pad 16: +5V -> N-0000060
Routing:
- net GND: track 0.00 -> 204.5 mm
- net +5V: track 0.00 -> 181.2 mm
- net +3.3V: track 0.00 -> 92.0 mm, vias 0 -> 1
- net N-0000033: track 0.00 -> 90.7 mm, vias 0 -> 1
- net N-0000045: track 0.00 -> 67.2 mm
- net N-0000022: track 0.00 -> 61.0 mm, vias 0 -> 1
- net N-0000017: track 0.00 -> 59.4 mm
- net N-0000016: track 0.00 -> 57.0 mm
- net N-0000019: track 0.00 -> 55.6 mm
- net N-0000015: track 0.00 -> 52.8 mm
- net N-0000013: track 0.00 -> 38.5 mm, vias 0 -> 1
- net N-0000031: track 0.00 -> 36.3 mm
- net N-0000056: track 0.00 -> 35.1 mm
- net N-0000032: track 0.00 -> 33.3 mm, vias 0 -> 1
- net N-0000054: track 0.00 -> 32.5 mm
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Other:
- board text added: "+5V"
