File: Circuit/hd44780_backpack.sch (KiCad schematic (older format))
At the start: 20 parts, among them IC1 ATTINY84A-SS, P1 I2C, P10 GND, P2 ISCP, P3 A0, P4 A1, P5 A7, P6 8, P7 10, P8 SERIAL QA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

Commit message: Added links to components
and prices to build a bom.
Parts:
- 10k1: Cost Per Unit (none) -> 0.77; Link (none) -> http://www.digikey.com.au/product-search/en?vendor=0&keywor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
- IC1: Cost Per Unit (none) -> 0.87
- SW1: Cost Per Unit (none) -> 0.1; Link (none) -> http://www.digikey.com.au/product-detail/en/FSM4JH/450-1650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
- U1: footprint ~ -> so-16; Cost per unit (none) -> 0.04
Changed lines of the file:
@@
 Sheet 1 1
 Title ""
-Date "13 may 2014"
+Date "7 jun 2014"
 Rev ""
 Comp ""
@@
 F 1 "ATTINY84A-SS" H 3150 1900 60  0000 C CNN
 F 2 "SO14" H 1950 1900 60  0001 C CNN
-F 3 "" H 2650 2650 60  0000 C CNN
+F 3 "http://www.atmel.com/Images/doc8006.pdf" H 2650 2650 60  0001 C CNN
+F 4 "0.87" H 2650 2650 60  0001 C CNN "Cost Per Unit"
 	1    2650 2650
 	1    0    0    -1
@@
 F 1 "POT" H 6450 1400 50  0000 C CNN
 F 2 "~" H 6450 1400 60  0000 C CNN
-F 3 "~" H 6450 1400 60  0000 C CNN
+F 3 "http://copal-electronics.info/en/00011/0064d.pdf" H 6450 1400 60  0001 C CNN
+F 4 "0.77" H 6450 1400 60  0001 C CNN "Cost Per Unit"
+F 5 "http://www.digikey.com.au/product-search/en?vendor=0&keywords=CT6EP103-ND" H 6450 1400 60  0001 C CNN "Link"
 	1    6450 1400
 	0    -1   -1   0
@@
 F 1 "Reset" H 3850 3620 50  0000 C CNN
 F 2 "~" H 3850 3700 60  0000 C CNN
-F 3 "~" H 3850 3700 60  0000 C CNN
+F 3 "http://www.te.com/commerce/DocumentDelivery/DDEController?Action=srchrtrv&DocNm=1825910&DocType=Customer+Drawing&DocLang=English" H 3850 3700 60  0001 C CNN
+F 4 "0.1" H 3850 3700 60  0001 C CNN "Cost Per Unit"
+F 5 "http://www.digikey.com.au/product-detail/en/FSM4JH/450-1650-ND/1632536" H 3850 3700 60  0001 C CNN "Link"
 	1    3850 3700
 	0    -1   -1   0
@@
 F 0 "U1" H 5400 4750 70  0000 C CNN
 F 1 "74HC595-16-PIN" H 5250 3550 70  0000 C CNN
-F 2 "~" H 5250 4150 60  0000 C CNN
-F 3 "~" H 5250 4150 60  0000 C CNN
+F 2 "so-16" H 5050 3700 60  0000 C CNN
+F 3 "http://www.nxp.com/documents/data_sheet/74HC_HCT595.pdf" H 5250 4150 60  0001 C CNN
+F 4 "0.04" H 5250 4150 60  0001 C CNN "Cost per unit"
 	1    5250 4150
 	1    0    0    -1
